Commit message: yobel recently updated [2024.08.12]

File: dyros_bolt_description/robots/bolt_with_passive-yobel.urdf (robot description, URDF)
Before this commit: robot dyros_bolt_description, 9 links, 8 joints
Links:
- link FL_FOOT: geometry collision mesh filename=../meshes/stl/bolt_foot.stl; visual mesh filename=../meshes/stl/bolt_foot.stl
- link FL_LOWER_LEG: geometry visual mesh filename=../meshes/stl/lower_leg_200mm_left_side.stl
- link FL_SHOULDER: geometry visual mesh filename=../meshes/stl/bolt_hip_fe_left_side.stl
- link FL_UPPER_LEG: geometry visual mesh filename=../meshes/stl/upper_leg_200mm_left_side.stl
- link FR_FOOT: geometry collision mesh filename=../meshes/stl/bolt_foot.stl; visual mesh filename=../meshes/stl/bolt_foot.stl
- link FR_LOWER_LEG: geometry visual mesh filename=../meshes/stl/lower_leg_200mm_right_side.stl
- link FR_SHOULDER: geometry visual mesh filename=../meshes/stl/bolt_hip_fe_right_side.stl
- link FR_UPPER_LEG: geometry visual mesh filename=../meshes/stl/upper_leg_200mm_right_side.stl
- link base_link: geometry collision sphere radius=0.18; visual mesh filename=../meshes/stl/bolt_body.stl

File: dyros_bolt_description/robots/bolt_with_passive.urdf (robot description, URDF)
Before this commit: robot bolt, 9 links, 8 joints
Joints:
- joint FL_ANKLE: limit lower=-10 upper=10 effort=1000 velocity=1000 -> lower=-1 upper=1 effort=2.5 velocity=20
- joint FL_HAA: limit lower=-10 upper=10 effort=1000 velocity=1000 -> lower=-0.36 upper=1.0472 effort=2.5 velocity=20
- joint FL_HFE: limit lower=-10 upper=10 effort=1000 velocity=1000 -> lower=-1.57 upper=1.57 effort=2.5 velocity=20
- joint FL_KFE: limit lower=-10 upper=10 effort=1000 velocity=1000 -> lower=-3.14 upper=0.0 effort=2.5 velocity=20
- joint FR_ANKLE: limit lower=-10 upper=10 effort=1000 velocity=1000 -> lower=-1 upper=1 effort=2.5 velocity=20
- joint FR_HAA: limit lower=-10 upper=10 effort=1000 velocity=1000 -> lower=-1.0472 upper=0.36 effort=2.5 velocity=20
- joint FR_HFE: limit lower=-10 upper=10 effort=1000 velocity=1000 -> lower=-1.57 upper=1.57 effort=2.5 velocity=20
- joint FR_KFE: limit lower=-10 upper=10 effort=1000 velocity=1000 -> lower=-3.14 upper=0.0 effort=2.5 velocity=20
